File: SensorBoard/SensorBoard.kicad_pcb (KiCad board)
At the start: 2 copper layers, 50.3 x 74 mm, 92 parts, among them U1 JST4Pin, U2 JST4Pin, U3 JST4Pin

Commit message: Added gerber files for SensorBoard and ArduinoBreakoutboard
Other:
- board text added: "Desingers: Jacob Kim, Olivia Wolfley, Chris Tran, Jorge Exinia,"
- board text added: "Mark I"
Changed lines of the file:
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@@
   (general
     (thickness 1.6)
-    (drawings 23)
+    (drawings 25)
     (tracks 108)
     (zones 0)
@@
   )
   (setup
-    (last_trace_width 0.5)
+    (last_trace_width 0.25)
     (user_trace_width 0.5)
     (user_trace_width 1.27)
@@
     (visible_elements 7FFFFFFF)
     (pcbplotparams
-      (layerselection 0x010fc_ffffffff)
+      (layerselection 0x3ffff_ffffffff)
       (usegerberextensions false)
       (usegerberattributes false)
       (usegerberadvancedattributes false)
-      (creategerberjobfile false)
+      (creategerberjobfile true)
       (excludeedgelayer true)
       (linewidth 0.100000)
@@
       (outputformat 1)
       (mirror false)
-      (drillshape 1)
+      (drillshape 0)
       (scaleselection 1)
-      (outputdirectory ""))
+      (outputdirectory "New folder/"))
   )
   (net 0 "")
@@
     )
   )
+  (gr_text "Mark  I" (at 169.545 110.109 270) (layer B.SilkS)
+    (effects (font (size 1 1) (thickness 0.15)) (justify mirror))
+  )
+  (gr_text "Desingers: Jacob Kim, Olivia Wolfley, Chris Tran, Jorge Exinia," (at 171.45 88.9 270) (layer B.SilkS)
+    (effects (font (size 1 1) (thickness 0.15)) (justify mirror))
+  )
   (gr_text Vin (at 169.545 81.153 90) (layer F.SilkS)
