File: Power Module/Power Module.sch (KiCad schematic (older format))
At the start: 4 parts, among them J1 Screw_Terminal_01x02, J3 Screw_Terminal_01x02, U1 LM2596

Commit message: Started work on v2 of Power Module
Updated and made schematic for v2 of power Module

Reworked PCB to address the new schematic
Parts:
- removed FUSE1: 64600001003, 646-SERIESHOLDER, symbol 64600001003:64600001003
- removed J3: Screw_Terminal_01x02, TerminalBlock_Phoenix:TerminalBlock_Phoenix_MKDS-3-2-5.08_1x02_P5.08mm_Horizontal, symbol Connector:Screw_Terminal_01x02
- added F1, F2, F3: 3A Fuse, 64600001003:646-SERIESHOLDER, symbol Device:Fuse
- added J2, J6: Screw_Terminal_01x02, TerminalBlock_MetzConnect:TerminalBlock_MetzConnect_Type094_RT03502HBLU_1x02_P5.00mm_Horizontal, symbol Connector:Screw_Terminal_01x02
- added J3, J4, J5: Conn_01x02, Connector_JST:JST_EH_B2B-EH-A_1x02_P2.50mm_Vertical, symbol Connector_Generic:Conn_01x02
- added U2, U3: LM2596, SCR_Parts_Library:LM2596, symbol SCR_KiCAD_Lib:LM2596
- J1: footprint TerminalBlock_Phoenix:TerminalBlock_Phoenix_MKDS-3-2-5.08_1x02_P5.08mm_Horizontal -> TerminalBlock_MetzConnect:TerminalBlock_MetzConnect_Type094_RT03502HBLU_1x02_P5.00mm_Horizontal
- U1: footprint SCR_KiCAD_Lib:LM2596 -> SCR_Parts_Library:LM2596
Connections:
- net labels added: +12V
- wire segments 16 -> 27
Other:
- note added: "3 Buck converters, in v2 all the power \nmodules are going on the same board.\nThis means we will need wide traces \nin the PCB."
- note added: "3 Screw terminals, 1 screw terminal will\n be for the 12V Battery in and the other \n2 will be for 12V out. One 12V out will\npower the motor controller, and the \nother will be for anything else"
- moved on the sheet: U1
