File: Arduino Breakout Board/ArduinoBreakoutboardControl.sch (KiCad schematic (older format))
At the start: 7 parts, among them M1 Conn_01x06_Male

Commit message: added an updated schematic with cleanner wire routing and updated the pcb for the schematic
Parts:
- removed IMU1: Conn_01x04_Male, Connector_JST:JST_EH_B4B-EH-A_1x04_P2.50mm_Vertical, symbol Connector:Conn_01x04_Male
- added U2: BNO-555, SCR_Parts_Library:BNO055, symbol bno-555:BNO-555
- renumbered ER1 to J1, EL1 to J2, M1 to J3, VOut1 to J4, Vin1 to J5, A1 to U1
Connections:
- net labels added: +5V, LeftB, RIghtA
- net labels removed: 5V, 5Vin, A, B, Vcc
- wire segments 69 -> 20
- no-connect marks 0 -> 20
Other:
- note added: "2 seperate JST Connecters both for \npowering and accessing 5 volts from the buck converter."
- note added: "5V"
- note added: "5Vin"
- note added: "ENA"
- note added: "ENB"
- note added: "GND"
- note added: "IMU Chip sending Gyroscope data to the\nmicroprocesser"
- note added: "IN1"
- note added: "IN2"
- note added: "IN3"
- note added: "IN4"
- note added: "JST Connector to send data \nto the motor controller. \n"
- note added: "JSTs to the motor encoders powering\n and sending data.\n"
- note added: "Left A"
- note added: "Left B"
- note added: "Right A"
- note added: "Right B"
- note added: "Vin"
- moved on the sheet: J1, J2, J3, J4, J5, U1

Commit message: started work on v2 of the Breakout board
Added Schematic for v2 of the Board

Updated PCB to address the changes done to the Schematic
Changed lines of the file:
@@
 Text Notes 3475 4175 0    50   ~ 0
 Left A
-Text Notes 3550 4875 0    50   ~ 0
+Text Notes 3550 4925 0    50   ~ 0
 ENA
-Text Notes 3550 4975 0    50   ~ 0
+Text Notes 3550 5025 0    50   ~ 0
 ENB
-Text Notes 3550 5075 0    50   ~ 0
+Text Notes 3550 5125 0    50   ~ 0
 IN1
-Text Notes 3550 5175 0    50   ~ 0
+Text Notes 3550 5225 0    50   ~ 0
 IN2
-Text Notes 3550 5275 0    50   ~ 0
+Text Notes 3550 5325 0    50   ~ 0
 IN3
-Text Notes 3550 5375 0    50   ~ 0
+Text Notes 3550 5425 0    50   ~ 0
 IN4
 Text Notes 8375 1575 0    50   ~ 0
@@
 Wire Wire Line
 	3925 3950 4325 3950
-Text GLabel 6375 4450 2    50   Input ~ 0
+Text GLabel 7275 4475 0    50   BiDi ~ 0
 SDA
-Text GLabel 7275 4475 0    50   Input ~ 0
-SDA
-Text GLabel 7275 4575 0    50   Input ~ 0
+Text GLabel 7275 4575 0    50   BiDi ~ 0
 SCL
-Text GLabel 6375 4650 2    50   Input ~ 0
+Text GLabel 6375 4650 2    50   BiDi ~ 0
 SCL
 NoConn ~ 7775 4075
@@
 Text GLabel 3900 4900 2    50   Input ~ 0
 ENA
-Text GLabel 5375 3950 0    50   Input ~ 0
+Text GLabel 5375 3950 0    50   Output ~ 0
 ENA
 Text GLabel 3900 5000 2    50   Input ~ 0
 ENB
-Text GLabel 5375 4050 0    50   Input ~ 0
+Text GLabel 5375 4050 0    50   Output ~ 0
 ENB
 Text GLabel 3900 5100 2    50   Input ~ 0
 IN1
-Text GLabel 5375 4250 0    50   Input ~ 0
+Text GLabel 5375 4250 0    50   Output ~ 0
 IN1
 Text GLabel 3900 5200 2    50   Input ~ 0
 IN2
-Text GLabel 5375 4350 0    50   Input ~ 0
+Text GLabel 5375 4350 0    50   Output ~ 0
 IN2
 Text GLabel 3900 5300 2    50   Input ~ 0
 IN3
-Text GLabel 5375 4450 0    50   Input ~ 0
+Text GLabel 5375 4450 0    50   Output ~ 0
 IN3
 Text GLabel 3900 5400 2    50   Input ~ 0
 IN4
-Text GLabel 5375 4650 0    50   Input ~ 0
+Text GLabel 5375 4650 0    50   Output ~ 0
 IN4
 Text Notes 3475 4275 0    50   ~ 0
 Left B
-Text GLabel 3925 3300 2    50   Input ~ 0
+Text GLabel 3925 3300 2    50   Output ~ 0
 RIghtA
-Text GLabel 3925 3400 2    50   Input ~ 0
+Text GLabel 3925 3400 2    50   Output ~ 0
 RightB
-Text GLabel 3925 4150 2    50   Input ~ 0
+Text GLabel 3925 4150 2    50   Output ~ 0
 LeftA
-Text GLabel 3925 4250 2    50   Input ~ 0
+Text GLabel 3925 4250 2    50   Output ~ 0
 LeftB
 NoConn ~ 6375 4050
@@
 	2900 3825 1425 3825
 NoConn ~ 5975 3050
+Text GLabel 6375 4450 2    50   BiDi ~ 0
+SDA
 $EndSCHEMATC

Commit message: added 2 more connectors for servos to the schematic and PCB
Updated and finished the PCB for V2
Parts:
- added J6, J7: Conn_01x03, Connector_JST:JST_EH_B3B-EH-A_1x03_P2.50mm_Vertical, symbol Connector_Generic:Conn_01x03
Connections:
- net labels added: +5VA, SERV1, SERV2
- wire segments 20 -> 21
- no-connect marks 20 -> 18
Other:
- note added: "Dpin1"
- note added: "Dpin2"
- note added: "JST connecttions for 2 servo motors \nfor the arm design, subject to change \nfor mechanical needs"
- moved on the sheet: J1, J2, J3

Commit message: Changed pins of the servo to PWM pins
deleted unneccesary schematic files
Changed lines of the file:
@@
 Text GLabel 3750 5925 2    50   Input ~ 0
-IN3
-Text GLabel 5375 4450 0    50   Output ~ 0
 IN3
 Text GLabel 3750 6025 2    50   Input ~ 0
@@
 Text GLabel 3825 2900 2    50   BiDi ~ 0
 SERV2
-Text GLabel 5375 4750 0    50   BiDi ~ 0
-SERV2
 Text GLabel 5375 4550 0    50   BiDi ~ 0
 SERV1
@@
 Wire Notes Line
 	1275 2700 1275 2425
+Text GLabel 5375 4450 0    50   BiDi ~ 0
+SERV2
+Text GLabel 5375 4750 0    50   Output ~ 0
+IN3
 $EndSCHEMATC
